Commit message: working on calibration parameters

File: ur_description/urdf/ur10.urdf.xacro (robot description, xacro)
@@ -27,10 +27,61 @@
   <!-- Kinematic model -->
   <!-- Properties from urcontrol.conf -->
-  <xacro:property name="ur10_d1" value="0.1273" />
-  <xacro:property name="ur10_a2" value="-0.612" />
-  <xacro:property name="ur10_a3" value="-0.5723" />
-  <xacro:property name="ur10_d4" value="0.163941" />
-  <xacro:property name="ur10_d5" value="0.1157" />
-  <xacro:property name="ur10_d6" value="0.0922" />
+  <property name="ur10_a1" value="0.0" />
+  <property name="ur10_a2" value="-0.612" />
+  <property name="ur10_a3" value="-0.5723" />
+  <property name="ur10_a4" value="0.0" />
+  <property name="ur10_a5" value="0.0" />
+  <property name="ur10_a5" value="0.0" />
+  <property name="ur10_d1" value="0.1273" />
+  <property name="ur10_d2" value="0.0" />
+  <property name="ur10_d3" value="0.0" />
+  <property name="ur10_d4" value="0.163941" />
+  <property name="ur10_d5" value="0.1157" />
+  <property name="ur10_d6" value="0.0922" />
+  <property name="ur10_alpha1" value="${pi / 2}" />
+  <property name="ur10_alpha2" value="0.0" />
+  <property name="ur10_alpha3" value="0.0" />
+  <property name="ur10_alpha4" value="${pi / 2}" />
+  <property name="ur10_alpha5" value="${-pi / 2}" />
+  <property name="ur10_alpha6" value="0.0" />
+  <!-- q_home_offset -->
+  <property name="ur10_theta1" value="0.0" />
+  <property name="ur10_theta2" value="${-pi / 2}" />
+  <property name="ur10_theta3" value="0.0" />
+  <property name="ur10_theta4" value="${-pi / 2}" />
+  <property name="ur10_theta5" value="0.0" />
+  <property name="ur10_theta6" value="0.0" />
+  <propery name="joint_direction_1" value="1.0" />
+  <propery name="joint_direction_2" value="1.0" />
+  <propery name="joint_direction_3" value="-1.0" />
+  <propery name="joint_direction_4" value="1.0" />
+  <propery name="joint_direction_5" value="1.0" />
+  <propery name="joint_direction_6" value="1.0" />
+  <!-- Calibrated model -->
+  <!-- Properties from calib.conf -->
+  <property name="delta_theta1" value="-0.0000197850701944219247" />
+  <property name="delta_theta2" value="0.000201462290104538797" />
+  <property name="delta_theta3" value="0.161845418395399482" />
+  <property name="delta_theta4" value="-0.161978431361046782" />
+  <property name="delta_theta5" value="-0.0000818201554555377376" />
+  <property name="delta_theta6" value="0.00000671758758682964541" />
+  <property name="delta_a1" value="0.000158446828127298446" />
+  <property name="delta_a2" value="-0.000365891870255152796" />
+  <property name="delta_a3" value="0.00859992418659250024" />
+  <property name="delta_a4" value="0.000185997155766058528" />
+  <property name="delta_a5" value="0.0000831112940804089751" />
+  <property name="delta_a5" value="0.0" />
+  <property name="delta_d1" value="0.000589172256288156282" />
+  <property name="delta_d2" value="-0.028897132408511942" />
+  <property name="delta_d3" value="-16.0423841961902234" />
+  <property name="delta_d4" value="16.0704712348591521" />
+  <property name="delta_d5" value="-0.0000989525525437184861" />
+  <property name="delta_d6" value="-0.000244457179784232648" />
+  <property name="delta_alpha1" value="0.000710613899062906285" />
+  <property name="delta_alpha2" value="-0.00296938046861772642" />
+  <property name="delta_alpha3" value="-0.00573144103189916678" />
+  <property name="delta_alpha4" value="-0.000192483211580940505" />
+  <property name="delta_alpha5" value="0.00030432728186813307" />
+  <property name="delta_alpha6" value="0.0" />
   <!-- Arbitrary offsets for shoulder/elbow joints -->
   <xacro:property name="shoulder_offset" value="0.220941" />  <!-- measured from model -->
@@ -80,5 +131,5 @@
       <parent link="${prefix}base_link" />
       <child link = "${prefix}shoulder_link" />
-      <origin xyz="0.0 0.0 ${shoulder_height}" rpy="0.0 0.0 0.0" />
+      <origin xyz="0.0 0.0 ${ur10_d1 + delta_d1}" rpy="0.0 0.0 0.0" />
       <axis xyz="0 0 1" />
       <xacro:unless value="${joint_limited}">

Commit message: cleaned up files for merge to master, reverted ur10.urdf.xacro to original state

File: ur_description/urdf/ur10.urdf.xacro (robot description, xacro)
@@ -27,62 +27,10 @@
   <!-- Kinematic model -->
   <!-- Properties from urcontrol.conf -->
-  <!-- When applying parameters keep in mind that the parameters are in CS base, not base_link, that is why some minuses appear -->
-  <property name="ur10_a1" value="0.0" />
-  <property name="ur10_a2" value="-0.612" />
-  <property name="ur10_a3" value="-0.5723" />
-  <property name="ur10_a4" value="0.0" />
-  <property name="ur10_a5" value="0.0" />
-  <property name="ur10_a6" value="0.0" />
-  <property name="ur10_d1" value="0.1273" />
-  <property name="ur10_d2" value="0.0" />
-  <property name="ur10_d3" value="0.0" />
-  <property name="ur10_d4" value="0.163941" />
-  <property name="ur10_d5" value="0.1157" />
-  <property name="ur10_d6" value="0.0922" />
-  <property name="ur10_alpha1" value="${pi / 2}" />
-  <property name="ur10_alpha2" value="0.0" />
-  <property name="ur10_alpha3" value="0.0" />
-  <property name="ur10_alpha4" value="${pi / 2}" />
-  <property name="ur10_alpha5" value="${-pi / 2}" />
-  <property name="ur10_alpha6" value="0.0" />
-  <!-- q_home_offset -->
-  <property name="ur10_theta1" value="0.0" />
-  <property name="ur10_theta2" value="${-pi / 2}" />
-  <property name="ur10_theta3" value="0.0" />
-  <property name="ur10_theta4" value="${-pi / 2}" />
-  <property name="ur10_theta5" value="0.0" />
-  <property name="ur10_theta6" value="0.0" />
-  <propery name="joint_direction_1" value="1.0" />
-  <propery name="joint_direction_2" value="1.0" />
-  <propery name="joint_direction_3" value="-1.0" />
-  <propery name="joint_direction_4" value="1.0" />
-  <propery name="joint_direction_5" value="1.0" />
-  <propery name="joint_direction_6" value="1.0" />
-  <!-- Calibrated model -->
-  <!-- Properties from calib.conf -->
-  <property name="delta_theta1" value="-0.0000197850701944219247" />
-  <property name="delta_theta2" value="0.000201462290104538797" />
-  <property name="delta_theta3" value="0.161845418395399482" />
-  <property name="delta_theta4" value="-0.161978431361046782" />
-  <property name="delta_theta5" value="-0.0000818201554555377376" />
-  <property name="delta_theta6" value="0.00000671758758682964541" />
-  <property name="delta_a1" value="0.000158446828127298446" />
-  <property name="delta_a2" value="-0.000365891870255152796" />
-  <property name="delta_a3" value="0.00859992418659250024" />
-  <property name="delta_a4" value="0.000185997155766058528" />
-  <property name="delta_a5" value="0.0000831112940804089751" />
-  <property name="delta_a5" value="0.0" />
-  <property name="delta_d1" value="0.000589172256288156282" />
-  <property name="delta_d2" value="-0.028897132408511942" />
-  <property name="delta_d3" value="-16.0423841961902234" />
-  <property name="delta_d4" value="16.0704712348591521" />
-  <property name="delta_d5" value="-0.0000989525525437184861" />
-  <property name="delta_d6" value="-0.000244457179784232648" />
-  <property name="delta_alpha1" value="0.000710613899062906285" />
-  <property name="delta_alpha2" value="-0.00296938046861772642" />
-  <property name="delta_alpha3" value="-0.00573144103189916678" />
-  <property name="delta_alpha4" value="-0.000192483211580940505" />
-  <property name="delta_alpha5" value="0.00030432728186813307" />
-  <property name="delta_alpha6" value="0.0" />
+  <xacro:property name="ur10_d1" value="0.1273" />
+  <xacro:property name="ur10_a2" value="-0.612" />
+  <xacro:property name="ur10_a3" value="-0.5723" />
+  <xacro:property name="ur10_d4" value="0.163941" />
+  <xacro:property name="ur10_d5" value="0.1157" />
+  <xacro:property name="ur10_d6" value="0.0922" />
   <!-- Arbitrary offsets for shoulder/elbow joints -->
   <xacro:property name="shoulder_offset" value="0.220941" />  <!-- measured from model -->
@@ -132,5 +80,5 @@
       <parent link="${prefix}base_link" />
       <child link = "${prefix}shoulder_link" />
-      <origin xyz="0.0 0.0 ${ur10_d1 + delta_d1}" rpy="0.0 0.0 ${delta_theta1}" />
+      <origin xyz="0.0 0.0 ${shoulder_height}" rpy="0.0 0.0 0.0" />
       <axis xyz="0 0 1" />
       <xacro:unless value="${joint_limited}">
@@ -163,5 +111,5 @@
       <parent link="${prefix}shoulder_link" />
       <child link = "${prefix}upper_arm_link" />
-      <origin xyz="0.0 0.0 0.0" rpy="0.0 ${-ur10_theta2} 0.0" />
+      <origin xyz="0.0 ${shoulder_offset} 0.0" rpy="0.0 ${pi / 2.0} 0.0" />
       <axis xyz="0 1 0" />
       <xacro:unless value="${joint_limited}">
@@ -194,5 +142,5 @@
       <parent link="${prefix}upper_arm_link" />
       <child link = "${prefix}forearm_link" />
-      <origin xyz="0.0 ${delta_d2} ${-ur10_a2-delta_a2}" rpy="0.0 ${delta_theta2} 0.0" />
+      <origin xyz="0.0 ${elbow_offset} ${upper_arm_length}" rpy="0.0 0.0 0.0" />
       <axis xyz="0 1 0" />
       <xacro:unless value="${joint_limited}">
@@ -225,5 +173,5 @@
       <parent link="${prefix}forearm_link" />
       <child link = "${prefix}wrist_1_link" />
-      <origin xyz="0.0 ${delta_d3} ${-ur10_a3-delta_a3}" rpy="0.0 ${pi / 2.0 + delta_theta3} 0.0" />
+      <origin xyz="0.0 0.0 ${forearm_length}" rpy="0.0 ${pi / 2.0} 0.0" />
       <axis xyz="0 1 0" />
       <xacro:unless value="${joint_limited}">
@@ -287,5 +235,5 @@
       <parent link="${prefix}wrist_2_link" />
       <child link = "${prefix}wrist_3_link" />
-      <origin xyz="0.0 0.0 ${ur10_d5+delta_d5}" rpy="0.0 0.0 0.0" />
+      <origin xyz="0.0 0.0 ${wrist_2_length}" rpy="0.0 0.0 0.0" />
       <axis xyz="0 1 0" />
       <xacro:unless value="${joint_limited}">
